File: KiCad/1_H-Board/H-Bridge_Proto.kicad_pcb (KiCad board)
At the start: 2 copper layers, 26.7 x 32.4 mm, 14 parts, among them J1 Conn_01x02, J2 Conn_01x02, J3 Conn_01x02, J4 Conn_01x02, J5 Conn_01x02, J6 Conn_01x03, U1 DRV8835

Commit message: Finished H-Bridge PCB V1
Parts:
- moved C5 2.95 mm to (135.1, 114.3)
- moved J1 1.27 mm to (128.3, 114.9)
- moved J2 1.27 mm to (128.3, 121.9)
- moved J5 1.27 mm to (128.3, 108.0)
- moved C4 1.21 mm to (135.1, 110.6)
- moved C2 1.20 mm to (130.0, 98.8)
- moved C3 0.92 mm to (137.0, 106.8)
- moved C1 0.63 mm to (137.0, 98.8)
- moved C6 0.52 mm to (135.1, 106.8)
Routing:
- net +8V: track 0.00 -> 33.4 mm
- net Net-(C5-Pad2): track 0.00 -> 19.9 mm
- net Net-(C5-Pad1): track 0.00 -> 18.2 mm
- net Net-(C4-Pad2): track 0.00 -> 14.4 mm
- net Net-(C4-Pad1): track 0.00 -> 12.8 mm
- net GND: track 4.97 -> 11.5 mm
- added copper zone on B.Cu, net GND
- added copper zone on F.Cu, net GND
Other:
- board size 26.7 x 32.4 mm -> 24.8 x 32.4 mm
- board text added: "H-Proto"
- board text added: "V1"
